Commit message: Update inertial parameters

File: ocs2_anymal_robot/urdf/anymal_gazebo.urdf.xacro (robot description, xacro)
@@ -96,5 +96,5 @@
     <plugin name="lf_contact_plugin" filename="libContactSensor.so"/>
     <contact>
-        <collision>fl_lleg_fixed_joint_lump__LF_FOOT_collision_sensor_collision</collision>
+        <collision>LF_SHANK_fixed_joint_lump__LF_FOOT_collision_sensor_collision_3</collision>
     </contact>
     </sensor>
@@ -104,5 +104,5 @@
     <plugin name="lh_contact_plugin" filename="libContactSensor.so"/>
     <contact>
-        <collision>hl_lleg_fixed_joint_lump__LH_FOOT_collision_sensor_collision</collision>
+        <collision>LH_SHANK_fixed_joint_lump__LH_FOOT_collision_sensor_collision_3</collision>
     </contact>
     </sensor>
@@ -112,5 +112,5 @@
     <plugin name="rf_contact_plugin" filename="libContactSensor.so"/>
     <contact>
-        <collision>fr_lleg_fixed_joint_lump__RF_FOOT_collision_sensor_collision</collision>
+        <collision>RF_SHANK_fixed_joint_lump__RF_FOOT_collision_sensor_collision_3</collision>
     </contact>
     </sensor>
@@ -120,5 +120,5 @@
     <plugin name="rh_contact_plugin" filename="libContactSensor.so"/>
     <contact>
-        <collision>hr_lleg_fixed_joint_lump__RH_FOOT_collision_sensor_collision</collision>
+        <collision>RH_SHANK_fixed_joint_lump__RH_FOOT_collision_sensor_collision_3</collision>
     </contact>
     </sensor>

File: ocs2_spot_robot/urdf/spot_gazebo.urdf.xacro (robot description, xacro)
@@ -356,5 +356,5 @@
     <plugin name="lf_contact_plugin" filename="libContactSensor.so"/>
     <contact>
-        <collision>fl_lleg_fixed_joint_lump__LF_FOOT_collision_sensor_collision</collision>
+        <collision>fl_lleg_fixed_joint_lump__LF_FOOT_collision_sensor_collision_1</collision>
     </contact>
     </sensor>
@@ -364,5 +364,5 @@
     <plugin name="lh_contact_plugin" filename="libContactSensor.so"/>
     <contact>
-        <collision>hl_lleg_fixed_joint_lump__LH_FOOT_collision_sensor_collision</collision>
+        <collision>hl_lleg_fixed_joint_lump__LH_FOOT_collision_sensor_collision_1</collision>
     </contact>
     </sensor>
@@ -372,5 +372,5 @@
     <plugin name="rf_contact_plugin" filename="libContactSensor.so"/>
     <contact>
-        <collision>fr_lleg_fixed_joint_lump__RF_FOOT_collision_sensor_collision</collision>
+        <collision>fr_lleg_fixed_joint_lump__RF_FOOT_collision_sensor_collision_1</collision>
     </contact>
     </sensor>
@@ -380,5 +380,5 @@
     <plugin name="rh_contact_plugin" filename="libContactSensor.so"/>
     <contact>
-        <collision>hr_lleg_fixed_joint_lump__RH_FOOT_collision_sensor_collision</collision>
+        <collision>hr_lleg_fixed_joint_lump__RH_FOOT_collision_sensor_collision_1</collision>
     </contact>
     </sensor>
