Commit message: adding camera to gripper, world for testing camera, simple script for visualizing image from new camera

File: ocs2_arm/urdf/spot_transmission.xacro (robot description, xacro)
@@ -4,5 +4,5 @@
         <transmission name="${name}">
             <type>transmission_interface/SimpleTransmission</type>
-            <joint name = "${joint}" >
+            <joint name="${joint}" >
                 <hardwareInterface>hardware_interface/EffortJointInterface</hardwareInterface>
             </joint>

File: ocs2_arm/urdf/spot_w_arm.urdf (robot description, URDF)
Before this commit: robot spot_w_arm, 26 links, 25 joints
Links:
- added link camera_link_arm, mass 1e-5
- added link camera_optical_arm, mass 1e-5
Joints:
- added joint camera: type fixed, parent gripper_1, child camera_link_arm, origin xyz=0.0 0.1 0.0 rpy=3.141592653589793 0.0 1.5707963267948966
- added joint camera_optical_joint_arm: type fixed, parent camera_link_arm, child camera_optical_arm, origin xyz=0.0 0.0 0.0 rpy=-1.57 0.0 -1.57
